File: IO.kicad_sch (KiCad schematic)
At the start: 9 parts, among them J6 JST_SH_1x6_SM06B-SRSS-TB-LF-SN, J7 JST_SH_1x6_SM06B-SRSS-TB-LF-SN

Commit message: [#71555] Remove dash from sch names
Other:
- title: audio-latency-processing-board -> Audio Latency Processing Board
Changed lines of the file:
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@@
 	(paper "A3")
 	(title_block
-		(title "audio-latency-processing-board")
+		(title "Audio Latency Processing Board")
 		(date "2025-01-07")
 		(rev "1.1.0")
