File: IO.kicad_sch (KiCad schematic)
At the start: 12 parts, among them J6 JST_SH_1x6_SM06B-SRSS-TB-LF-SN, J7 JST_SH_1x6_SM06B-SRSS-TB-LF-SN, U13 TPD4E05U06QDQARQ1, U14 TPD4E05U06QDQARQ1

Commit message: [#77779] Rename to audio latency tester board
Other:
- title: Audio controller board -> Audio latency tester board
Changed lines of the file:
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@@
 	(paper "A3")
 	(title_block
-		(title "Audio controller board")
+		(title "Audio latency tester board")
 		(date "2025-04-03")
 		(rev "1.3.2")
@@
 		)
 		(instances
-			(project "audio-controller-board"
+			(project "audio-latency-tester-board"
 				(path "/7fb12ebf-f685-4412-b638-445b1bf344bc/1277d361-8469-440e-97d3-29bbfd6c9b73"
 					(reference "#PWR0132")
@@
 		)
 		(instances
-			(project "audio-controller-board"
+			(project "audio-latency-tester-board"
 				(path "/7fb12ebf-f685-4412-b638-445b1bf344bc/1277d361-8469-440e-97d3-29bbfd6c9b73"
 					(reference "#PWR035")
@@
 		)
 		(instances
-			(project "audio-controller-board"
+			(project "audio-latency-tester-board"
 				(path "/7fb12ebf-f685-4412-b638-445b1bf344bc/1277d361-8469-440e-97d3-29bbfd6c9b73"
 					(reference "#PWR04")
@@
 		)
 		(instances
-			(project "audio-controller-board"
+			(project "audio-latency-tester-board"
 				(path "/7fb12ebf-f685-4412-b638-445b1bf344bc/1277d361-8469-440e-97d3-29bbfd6c9b73"
 					(reference "R88")
@@
 		)
 		(instances
-			(project "audio-controller-board"
+			(project "audio-latency-tester-board"
 				(path "/7fb12ebf-f685-4412-b638-445b1bf344bc/1277d361-8469-440e-97d3-29bbfd6c9b73"
 					(reference "#PWR0134")
@@
 		)
 		(instances
-			(project "audio-controller-board"
+			(project "audio-latency-tester-board"
 				(path "/7fb12ebf-f685-4412-b638-445b1bf344bc/1277d361-8469-440e-97d3-29bbfd6c9b73"
 					(reference "#PWR0125")
@@
 		)
 		(instances
-			(project "audio-controller-board"
+			(project "audio-latency-tester-board"
 				(path "/7fb12ebf-f685-4412-b638-445b1bf344bc/1277d361-8469-440e-97d3-29bbfd6c9b73"
 					(reference "U14")
@@
 		)
 		(instances
-			(project "audio-controller-board"
+			(project "audio-latency-tester-board"
 				(path "/7fb12ebf-f685-4412-b638-445b1bf344bc/1277d361-8469-440e-97d3-29bbfd6c9b73"
 					(reference "J7")
@@
 		)
 		(instances
-			(project "audio-controller-board"
+			(project "audio-latency-tester-board"
 				(path "/7fb12ebf-f685-4412-b638-445b1bf344bc/1277d361-8469-440e-97d3-29bbfd6c9b73"
 					(reference "#PWR0126")
@@
 		)
 		(instances
-			(project "audio-controller-board"
+			(project "audio-latency-tester-board"
 				(path "/7fb12ebf-f685-4412-b638-445b1bf344bc/1277d361-8469-440e-97d3-29bbfd6c9b73"
 					(reference "R3")
@@
 		)
 		(instances
-			(project "audio-controller-board"
+			(project "audio-latency-tester-board"
 				(path "/7fb12ebf-f685-4412-b638-445b1bf344bc/1277d361-8469-440e-97d3-29bbfd6c9b73"
 					(reference "D8")
@@
 		)
 		(instances
-			(project "audio-controller-board"
+			(project "audio-latency-tester-board"
 				(path "/7fb12ebf-f685-4412-b638-445b1bf344bc/1277d361-8469-440e-97d3-29bbfd6c9b73"
 					(reference "#PWR0151")
@@
 		)
 		(instances
-			(project "audio-controller-board"
+			(project "audio-latency-tester-board"
 				(path "/7fb12ebf-f685-4412-b638-445b1bf344bc/1277d361-8469-440e-97d3-29bbfd6c9b73"
 					(reference "#PWR0124")
@@
 		)
 		(instances
-			(project "audio-controller-board"
+			(project "audio-latency-tester-board"
 				(path "/7fb12ebf-f685-4412-b638-445b1bf344bc/1277d361-8469-440e-97d3-29bbfd6c9b73"
 					(reference "R87")
@@
 		)
 		(instances
-			(project "audio-controller-board"
+			(project "audio-latency-tester-board"
 				(path "/7fb12ebf-f685-4412-b638-445b1bf344bc/1277d361-8469-440e-97d3-29bbfd6c9b73"
 					(reference "#PWR0135")
@@
 		)
 		(instances
-			(project "audio-controller-board"
+			(project "audio-latency-tester-board"
 				(path "/7fb12ebf-f685-4412-b638-445b1bf344bc/1277d361-8469-440e-97d3-29bbfd6c9b73"
 					(reference "U13")
@@
 		)
 		(instances
-			(project "audio-controller-board"
+			(project "audio-latency-tester-board"
 				(path "/7fb12ebf-f685-4412-b638-445b1bf344bc/1277d361-8469-440e-97d3-29bbfd6c9b73"
 					(reference "#PWR0133")
@@
 		)
 		(instances
-			(project "audio-controller-board"
+			(project "audio-latency-tester-board"
 				(path "/7fb12ebf-f685-4412-b638-445b1bf344bc/1277d361-8469-440e-97d3-29bbfd6c9b73"
 					(reference "D4")
@@
 		)
 		(instances
-			(project "audio-controller-board"
+			(project "audio-latency-tester-board"
 				(path "/7fb12ebf-f685-4412-b638-445b1bf344bc/1277d361-8469-440e-97d3-29bbfd6c9b73"
 					(reference "#PWR0152")
@@
 		)
 		(instances
-			(project "audio-controller-board"
+			(project "audio-latency-tester-board"
 				(path "/7fb12ebf-f685-4412-b638-445b1bf344bc/1277d361-8469-440e-97d3-29bbfd6c9b73"
 					(reference "#PWR0150")
@@
 		)
 		(instances
-			(project "audio-controller-board"
+			(project "audio-latency-tester-board"
 				(path "/7fb12ebf-f685-4412-b638-445b1bf344bc/1277d361-8469-440e-97d3-29bbfd6c9b73"
 					(reference "C55")
@@
 		)
 		(instances
-			(project "audio-controller-board"
+			(project "audio-latency-tester-board"
 				(path "/7fb12ebf-f685-4412-b638-445b1bf344bc/1277d361-8469-440e-97d3-29bbfd6c9b73"
 					(reference "#PWR02")
