File: Mic_Conn.kicad_sch (KiCad schematic)
At the start: 18 parts, among them J1 Conn_FFC_Molex_5019510550, J2 Conn_FFC_Molex_5019510550, J8 JST_SUR_1x5_BM05B-SURS-TB-LF-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, U1 TPD4E05U06QDQARQ1, U4 TPD4E02B04DQA, U6 TPD4E05U06QDQARQ1

Commit message: [#77779] Rename to audio latency tester board
Other:
- title: Audio controller board -> Audio latency tester board
Changed lines of the file:
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@@
 	(paper "A3")
 	(title_block
-		(title "Audio controller board")
+		(title "Audio latency tester board")
 		(date "2025-04-03")
 		(rev "1.3.2")
@@
 		)
 		(instances
-			(project "audio-controller-board"
+			(project "audio-latency-tester-board"
 				(path "/7fb12ebf-f685-4412-b638-445b1bf344bc/a5973bba-065b-4f1e-8188-1e9f006e3cba"
 					(reference "R22")
@@
 		)
 		(instances
-			(project "audio-controller-board"
+			(project "audio-latency-tester-board"
 				(path "/7fb12ebf-f685-4412-b638-445b1bf344bc/a5973bba-065b-4f1e-8188-1e9f006e3cba"
 					(reference "#PWR05")
@@
 		)
 		(instances
-			(project "audio-controller-board"
+			(project "audio-latency-tester-board"
 				(path "/7fb12ebf-f685-4412-b638-445b1bf344bc/a5973bba-065b-4f1e-8188-1e9f006e3cba"
 					(reference "R18")
@@
 		)
 		(instances
-			(project "audio-controller-board"
+			(project "audio-latency-tester-board"
 				(path "/7fb12ebf-f685-4412-b638-445b1bf344bc/a5973bba-065b-4f1e-8188-1e9f006e3cba"
 					(reference "#PWR027")
@@
 		)
 		(instances
-			(project "audio-controller-board"
+			(project "audio-latency-tester-board"
 				(path "/7fb12ebf-f685-4412-b638-445b1bf344bc/a5973bba-065b-4f1e-8188-1e9f006e3cba"
 					(reference "#PWR0148")
@@
 		)
 		(instances
-			(project "audio-controller-board"
+			(project "audio-latency-tester-board"
 				(path "/7fb12ebf-f685-4412-b638-445b1bf344bc/a5973bba-065b-4f1e-8188-1e9f006e3cba"
 					(reference "C4")
@@
 		)
 		(instances
-			(project "audio-controller-board"
+			(project "audio-latency-tester-board"
 				(path "/7fb12ebf-f685-4412-b638-445b1bf344bc/a5973bba-065b-4f1e-8188-1e9f006e3cba"
 					(reference "#PWR03")
@@
 		)
 		(instances
-			(project "audio-controller-board"
+			(project "audio-latency-tester-board"
 				(path "/7fb12ebf-f685-4412-b638-445b1bf344bc/a5973bba-065b-4f1e-8188-1e9f006e3cba"
 					(reference "#PWR040")
@@
 		)
 		(instances
-			(project "audio-controller-board"
+			(project "audio-latency-tester-board"
 				(path "/7fb12ebf-f685-4412-b638-445b1bf344bc/a5973bba-065b-4f1e-8188-1e9f006e3cba"
 					(reference "R21")
@@
 		)
 		(instances
-			(project "audio-controller-board"
+			(project "audio-latency-tester-board"
 				(path "/7fb12ebf-f685-4412-b638-445b1bf344bc/a5973bba-065b-4f1e-8188-1e9f006e3cba"
 					(reference "#PWR0147")
@@
 		)
 		(instances
-			(project "audio-controller-board"
+			(project "audio-latency-tester-board"
 				(path "/7fb12ebf-f685-4412-b638-445b1bf344bc/a5973bba-065b-4f1e-8188-1e9f006e3cba"
 					(reference "#PWR023")
@@
 		)
 		(instances
-			(project "audio-controller-board"
+			(project "audio-latency-tester-board"
 				(path "/7fb12ebf-f685-4412-b638-445b1bf344bc/a5973bba-065b-4f1e-8188-1e9f006e3cba"
 					(reference "C5")
@@
 		)
 		(instances
-			(project "audio-controller-board"
+			(project "audio-latency-tester-board"
 				(path "/7fb12ebf-f685-4412-b638-445b1bf344bc/a5973bba-065b-4f1e-8188-1e9f006e3cba"
 					(reference "R4")
@@
 		)
 		(instances
-			(project "audio-controller-board"
+			(project "audio-latency-tester-board"
 				(path "/7fb12ebf-f685-4412-b638-445b1bf344bc/a5973bba-065b-4f1e-8188-1e9f006e3cba"
 					(reference "C56")
@@
 		)
 		(instances
-			(project "audio-controller-board"
+			(project "audio-latency-tester-board"
 				(path "/7fb12ebf-f685-4412-b638-445b1bf344bc/a5973bba-065b-4f1e-8188-1e9f006e3cba"
 					(reference "J2")
@@
 		)
 		(instances
-			(project "audio-controller-board"
+			(project "audio-latency-tester-board"
 				(path "/7fb12ebf-f685-4412-b638-445b1bf344bc/a5973bba-065b-4f1e-8188-1e9f006e3cba"
 					(reference "J8")
@@
 		)
 		(instances
-			(project "audio-controller-board"
+			(project "audio-latency-tester-board"
 				(path "/7fb12ebf-f685-4412-b638-445b1bf344bc/a5973bba-065b-4f1e-8188-1e9f006e3cba"
 					(reference "R93")
@@
 		)
 		(instances
-			(project "audio-controller-board"
+			(project "audio-latency-tester-board"
 				(path "/7fb12ebf-f685-4412-b638-445b1bf344bc/a5973bba-065b-4f1e-8188-1e9f006e3cba"
 					(reference "U6")
@@
 		)
 		(instances
-			(project "audio-controller-board"
+			(project "audio-latency-tester-board"
 				(path "/7fb12ebf-f685-4412-b638-445b1bf344bc/a5973bba-065b-4f1e-8188-1e9f006e3cba"
 					(reference "R25")
@@
 		)
 		(instances
-			(project "audio-controller-board"
+			(project "audio-latency-tester-board"
 				(path "/7fb12ebf-f685-4412-b638-445b1bf344bc/a5973bba-065b-4f1e-8188-1e9f006e3cba"
 					(reference "#PWR0143")
@@
 		)
 		(instances
-			(project "audio-controller-board"
+			(project "audio-latency-tester-board"
 				(path "/7fb12ebf-f685-4412-b638-445b1bf344bc/a5973bba-065b-4f1e-8188-1e9f006e3cba"
 					(reference "#PWR024")
@@
 		)
 		(instances
-			(project "audio-controller-board"
+			(project "audio-latency-tester-board"
 				(path "/7fb12ebf-f685-4412-b638-445b1bf344bc/a5973bba-065b-4f1e-8188-1e9f006e3cba"
 					(reference "R24")
@@
 		)
 		(instances
-			(project "audio-controller-board"
+			(project "audio-latency-tester-board"
 				(path "/7fb12ebf-f685-4412-b638-445b1bf344bc/a5973bba-065b-4f1e-8188-1e9f006e3cba"
 					(reference "#PWR025")
@@
 		)
 		(instances
-			(project "audio-controller-board"
+			(project "audio-latency-tester-board"
 				(path "/7fb12ebf-f685-4412-b638-445b1bf344bc/a5973bba-065b-4f1e-8188-1e9f006e3cba"
 					(reference "R23")
@@
 		)
 		(instances
-			(project "audio-controller-board"
+			(project "audio-latency-tester-board"
 				(path "/7fb12ebf-f685-4412-b638-445b1bf344bc/a5973bba-065b-4f1e-8188-1e9f006e3cba"
 					(reference "U4")
@@
 		)
 		(instances
-			(project "audio-controller-board"
+			(project "audio-latency-tester-board"
 				(path "/7fb12ebf-f685-4412-b638-445b1bf344bc/a5973bba-065b-4f1e-8188-1e9f006e3cba"
 					(reference "R20")
@@
 		)
 		(instances
-			(project "audio-controller-board"
+			(project "audio-latency-tester-board"
 				(path "/7fb12ebf-f685-4412-b638-445b1bf344bc/a5973bba-065b-4f1e-8188-1e9f006e3cba"
 					(reference "#PWR026")
